File: KiCad/KS0835F.sch (KiCad schematic (older format))
At the start: 48 parts, among them Q1 2N7000, U3 4050, U4 KS0835F, U5 LM358

Commit message: Add files via upload
Parts:
- D4: footprint Diode_THT:D_DO-41_SOD81_P10.16mm_Horizontal -> Diode_THT:D_DO-15_P10.16mm_Horizontal
Changed lines of the file:
@@
 F 0 "D4" H 3700 1975 50  0000 C CNN
 F 1 "P6KE82" H 3700 1725 50  0000 C CNN
-F 2 "Diode_THT:D_DO-41_SOD81_P10.16mm_Horizontal" H 3700 1850 50  0001 C CNN
+F 2 "Diode_THT:D_DO-15_P10.16mm_Horizontal" H 3700 1850 50  0001 C CNN
 F 3 "~" H 3700 1850 50  0001 C CNN
 	1    3700 1850
